Commit message: fixed indentation issues; moved files to correct folders

File: models/hokuyo/hokuyo.xacro (robot description, xacro)
@@ -1,46 +1,46 @@
 <?xml version="1.0"?>
 <robot xmlns:xacro="http://ros.org/wiki/xacro">
-	<!-- Laser Sensor Defintion -->
+  <!-- Laser Sensor Defintion -->
   <link name="${laser_name}">
-	  <gravity>false</gravity>
-	  <inertial>
-		  <mass value="0.0001"/>
-		  <origin xyz="0 0 0"/>
-		  <inertia ixx="1" ixy="0" ixz="0"
-				   iyy="1" iyz="0" izz="1"/>
-	  </inertial>
-	  <visual name="visual">
-	    <geometry>
-			<mesh filename="model://hokuyo/meshes/hokuyo.dae"/>
-	    </geometry>
-	  </visual>
+    <gravity>false</gravity>
+	<inertial>
+	  <mass value="0.0001"/>
+	  <origin xyz="0 0 0"/>
+	  <inertia ixx="1" ixy="0" ixz="0"
+			   iyy="1" iyz="0" izz="1"/>
+	</inertial>
+	<visual name="visual">
+	  <geometry>
+	    <mesh filename="model://hokuyo/meshes/hokuyo.dae"/>
+	  </geometry>
+	</visual>
   </link>
   <gazebo reference="${laser_name}">
 	<sensor name="${laser_name}" type="ray">
-	    <visualize>true</visualize>
-	    <ray>
-	      <scan>
-	        <horizontal>
-	          <samples>640</samples>
-	          <resolution>1</resolution>
-	          <min_angle>-1</min_angle>
-	          <max_angle>1</max_angle>
-	        </horizontal>
-	      </scan>
-	      <range>
-	        <min>0.08</min>
-	        <max>10</max>
-	        <resolution>0.01</resolution>
-	      </range>
-	    </ray>
-	    <plugin name="${laser_name}" filename="libgazebo_ros_laser.so" >
-	    	<always_on>true</always_on>
-	    	<updateRate>0.0</updateRate>
-	    	<topicName>${publish_topic}</topicName>
-	    </plugin>
-	    <always_on>1</always_on>
-	    <update_rate>30</update_rate>
-	    <visualize>true</visualize>
-	  </sensor>
+	  <visualize>true</visualize>
+	  <ray>
+	    <scan>
+	      <horizontal>
+	        <samples>640</samples>
+	        <resolution>1</resolution>
+	        <min_angle>-1</min_angle>
+	        <max_angle>1</max_angle>
+	      </horizontal>
+	    </scan>
+	    <range>
+	      <min>0.08</min>
+	      <max>10</max>
+	      <resolution>0.01</resolution>
+	    </range>
+	  </ray>
+	  <plugin name="${laser_name}" filename="libgazebo_ros_laser.so" >
+	    <always_on>true</always_on>
+	    <updateRate>0.0</updateRate>
+	    <topicName>${publish_topic}</topicName>
+	  </plugin>
+	  <always_on>1</always_on>
+	  <update_rate>30</update_rate>
+	  <visualize>true</visualize>
+	</sensor>
   </gazebo>
   <joint name="${laser_name}_joint" type="fixed">

Commit message: Created map in .pgm and .yaml form

File: models/hokuyo/hokuyo.xacro (robot description, xacro)
@@ -24,6 +24,6 @@
 	        <samples>640</samples>
 	        <resolution>1</resolution>
-	        <min_angle>-1</min_angle>
-	        <max_angle>1</max_angle>
+	        <min_angle>-${scan_angle}</min_angle>
+	        <max_angle>${scan_angle}</max_angle>
 	      </horizontal>
 	    </scan>
@@ -36,6 +36,7 @@
 	  <plugin name="${laser_name}" filename="libgazebo_ros_laser.so" >
 	    <always_on>true</always_on>
-	    <updateRate>0.0</updateRate>
+	    <updateRate>100.0</updateRate>
 	    <topicName>${publish_topic}</topicName>
+	    <frameName>${frame_id}</frameName>
 	  </plugin>
 	  <always_on>1</always_on>
@@ -46,5 +47,5 @@
   <joint name="${laser_name}_joint" type="fixed">
 	<origin xyz="${xyz}" rpy="${rpy}"/>
-	<parent link="base_link"/>
+	<parent link="${parent_link}"/>
 	<child link="${laser_name}"/>
   </joint>

File: models/p3dx_with_sensors/pioneer3dx.xacro (robot description, xacro)
@@ -4,13 +4,19 @@
   <!-- Front Laser -->
   <xacro:property name="laser_name" value="front_laser"/>
+  <xacro:property name="parent_link" value="base_link"/>
+  <xacro:property name="frame_id" value="pioneer/front_laser"/>
   <xacro:property name="xyz" value="0.1 0 0.3"/>
   <xacro:property name="rpy" value="0 0 0"/>
-  <xacro:property name="publish_topic" value="scan_front"/>
+  <xacro:property name="publish_topic" value="pioneer/front_laser"/>
+  <xacro:property name="scan_angle" value="2.36"/>
   <xacro:include filename="$(find ariac_environment)/models/hokuyo/hokuyo.xacro"/>
   <!-- Back Laser -->
   <xacro:property name="laser_name" value="back_laser"/>
+  <xacro:property name="parent_link" value="base_link"/>
+  <xacro:property name="frame_id" value="pioneer/back_laser"/>
   <xacro:property name="xyz" value="-0.2 0 0.3"/>
   <xacro:property name="rpy" value="0 0 3.14"/>
-  <xacro:property name="publish_topic" value="scan_back"/>
+  <xacro:property name="publish_topic" value="pioneer/back_laser"/>
+  <xacro:property name="scan_angle" value="2.36"/>
   <xacro:include filename="$(find ariac_environment)/models/hokuyo/hokuyo.xacro"/>
 </robot>

Commit message: Add fake localization. Closes #8.
- also add proper node namespacing
- fix Hokuyo urdf (provide package name in mesh URL)

File: models/hokuyo/hokuyo.xacro (robot description, xacro)
@@ -12,5 +12,5 @@
 	<visual name="visual">
 	  <geometry>
-	    <mesh filename="model://hokuyo/meshes/hokuyo.dae"/>
+	    <mesh filename="package://ariac_environment/models/hokuyo/meshes/hokuyo.dae"/>
 	  </geometry>
 	</visual>
